File: WeMos D1 mini.sch (EAGLE design)
At the start: 19 parts

Commit message: Changed esp8266modules.lbr (esthetics)
Parts:
- renumbered WEMOS1 to _
Changed lines of the file:
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@@
 </classes>
 <parts>
-<part name="WEMOS1" library="esp8266modules" deviceset="WEMOS-D1-MINI" device=""/>
+<part name="_" library="esp8266modules" deviceset="WEMOS-D1-MINI" device=""/>
 <part name="S1" library="switch-omron" library_urn="urn:adsk.eagle:library:377" deviceset="10-XX" device="" package3d_urn="urn:adsk.eagle:package:27496/1"/>
 <part name="S2" library="switch-omron" library_urn="urn:adsk.eagle:library:377" deviceset="10-XX" device="" package3d_urn="urn:adsk.eagle:package:27496/1"/>
@@
 </plain>
 <instances>
-<instance part="WEMOS1" gate="D1" x="20.32" y="55.88"/>
+<instance part="_" gate="D1" x="20.32" y="55.88"/>
 <instance part="S1" gate="1" x="81.28" y="71.12" rot="R270"/>
 <instance part="S2" gate="1" x="96.52" y="71.12" rot="R270"/>
@@
 <net name="VCC" class="1">
 <segment>
-<pinref part="WEMOS1" gate="D1" pin="3V3"/>
+<pinref part="_" gate="D1" pin="3V3"/>
 <wire x1="5.08" y1="48.26" x2="-5.08" y2="48.26" width="0.1524" layer="91"/>
 <label x="-5.08" y="48.26" size="1.778" layer="95"/>
@@
 <wire x1="86.36" y1="50.8" x2="101.6" y2="50.8" width="0.1524" layer="91"/>
 <wire x1="86.36" y1="68.58" x2="86.36" y2="50.8" width="0.1524" layer="91"/>
-<pinref part="WEMOS1" gate="D1" pin="GND"/>
+<pinref part="_" gate="D1" pin="GND"/>
 <wire x1="38.1" y1="50.8" x2="86.36" y2="50.8" width="0.1524" layer="91"/>
 <junction x="86.36" y="50.8"/>
@@
 <net name="D5" class="0">
 <segment>
-<pinref part="WEMOS1" gate="D1" pin="D5"/>
+<pinref part="_" gate="D1" pin="D5"/>
 <wire x1="5.08" y1="58.42" x2="-5.08" y2="58.42" width="0.1524" layer="91"/>
 <label x="-5.08" y="58.42" size="1.778" layer="95"/>
@@
 <net name="D6" class="0">
 <segment>
-<pinref part="WEMOS1" gate="D1" pin="D6"/>
+<pinref part="_" gate="D1" pin="D6"/>
 <wire x1="5.08" y1="55.88" x2="-5.08" y2="55.88" width="0.1524" layer="91"/>
 <label x="-5.08" y="55.88" size="1.778" layer="95"/>
@@
 <net name="D7" class="0">
 <segment>
-<pinref part="WEMOS1" gate="D1" pin="D7"/>
+<pinref part="_" gate="D1" pin="D7"/>
 <wire x1="-5.08" y1="53.34" x2="5.08" y2="53.34" width="0.1524" layer="91"/>
 <label x="-5.08" y="53.34" size="1.778" layer="95"/>
@@
 <net name="D4" class="0">
 <segment>
-<pinref part="WEMOS1" gate="D1" pin="D4"/>
+<pinref part="_" gate="D1" pin="D4"/>
 <wire x1="38.1" y1="53.34" x2="50.8" y2="53.34" width="0.1524" layer="91"/>
 <label x="45.72" y="53.34" size="1.778" layer="95"/>
@@
 <net name="D3" class="0">
 <segment>
-<pinref part="WEMOS1" gate="D1" pin="D3"/>
+<pinref part="_" gate="D1" pin="D3"/>
 <wire x1="38.1" y1="55.88" x2="50.8" y2="55.88" width="0.1524" layer="91"/>
 <label x="48.26" y="55.88" size="1.778" layer="95"/>
@@
 <net name="D2" class="0">
 <segment>
-<pinref part="WEMOS1" gate="D1" pin="D2"/>
+<pinref part="_" gate="D1" pin="D2"/>
 <wire x1="38.1" y1="58.42" x2="50.8" y2="58.42" width="0.1524" layer="91"/>
 <label x="45.72" y="58.42" size="1.778" layer="95"/>
@@
 <net name="D0" class="0">
 <segment>
-<pinref part="WEMOS1" gate="D1" pin="D0"/>
+<pinref part="_" gate="D1" pin="D0"/>
 <wire x1="5.08" y1="60.96" x2="-5.08" y2="60.96" width="0.1524" layer="91"/>
 <label x="-5.08" y="60.96" size="1.778" layer="95"/>
@@
 <net name="A0" class="0">
 <segment>
-<pinref part="WEMOS1" gate="D1" pin="A0"/>
+<pinref part="_" gate="D1" pin="A0"/>
 <wire x1="5.08" y1="63.5" x2="-5.08" y2="63.5" width="0.1524" layer="91"/>
 <label x="-5.08" y="63.5" size="1.778" layer="95"/>
@@
 <net name="D1" class="0">
 <segment>
-<pinref part="WEMOS1" gate="D1" pin="D1"/>
+<pinref part="_" gate="D1" pin="D1"/>
 <wire x1="38.1" y1="60.96" x2="50.8" y2="60.96" width="0.1524" layer="91"/>
 <label x="45.72" y="60.96" size="1.778" layer="95"/>
@@
 <net name="D8" class="0">
 <segment>
-<pinref part="WEMOS1" gate="D1" pin="D8"/>
+<pinref part="_" gate="D1" pin="D8"/>
 <wire x1="5.08" y1="50.8" x2="-5.08" y2="50.8" width="0.1524" layer="91"/>
 <label x="-5.08" y="50.8" size="1.778" layer="95"/>

Commit message: 1st prototype candidate 1
Parts:
- added GND: (no value), pinhead_v2:PINHD-1X4/OCT
- added LED1: (no value), led:LED3MM
- added R1: (no value), resistor:R-EU_0204/5
- JP1: device pinhead_v2:PINHD-1X6/OCT -> pinhead_v2:PINHD-1X7/OCT
- R6: value (none) -> 10K
- renumbered JP2 to VCC, JP4 to GND-VCC-GND
Connections:
- new net N$6: LED0.A, R0.1
- net A0: no longer JP1.3
- net D0: now also JP1.1, R0.2; no longer JP1.4, LED0.A
- net D1: now also JP1.2, R1.2; no longer JP1.5
- net D2: now also JP1.3, R2.2; no longer JP1.6, LED2.A
- net D3: now also JP1.4, R3.2; no longer LED3.A
- net D4: now also JP1.5, R4.2; no longer LED4.A
- net D5: now also JP1.6, R5.2; no longer LED5.A
- net D6: now also JP1.7
- net GND: now also GND.1, GND.2, GND.3, GND.4, LED0.C, LED1.C, LED2.C, LED3.C, LED4.C, LED5.C; no longer JP1.1, JP1.2, R0.1, R2.1, R3.1, R4.1, R5.1
- net N$1: now also LED5.A, R5.1; no longer LED0.C, R0.2
- net N$2: now also LED4.A, R4.1; no longer LED2.C, R2.2
- net N$3: now also LED3.A, R3.1; no longer LED3.C, R3.2
- net N$4: now also LED2.A, R2.1; no longer LED4.C, R4.2
- net N$5: now also LED1.A, R1.1; no longer LED5.C, R5.2
Other:
- note removed: "D1 is reserved for relay module"
- moved on the sheet: LED0, LED2, LED3, LED4, LED5, R0, R2, R3, R4, R5

Commit message: https://PCBs.io/share/z5oeo
Parts:
- removed S1, S2: (no value), switch-omron:10-XX
- added BTN7: GND-D7, pinhead_v2:PINHD-1X2/OCT
- added BTN8: GND-D8, pinhead_v2:PINHD-1X2/OCT
- added RA0: 10K, resistor:R-EU_0204/5
- added VCC-GND-5V: (no value), pinhead_v2:PINHD-1X3/OCT
- JP1: device pinhead_v2:PINHD-1X7/OCT -> pinhead_v2:PINHD-1X8/OCT
- JP3: value (none) -> A0-D0-D1-D2-D3; device pinhead_v2:PINHD-1X4/OCT -> pinhead_v2:PINHD-1X5/OCT
- TMP: value (none) -> VCC-D6-GND
Connections:
- new net 5V: VCC-GND-5V.3, _.5V
- net A0: now also RA0.2
- net D3: now also JP3.5
- net D6: no longer JP1.7
- net D7: now also BTN7.1, JP1.7; no longer S1.P, S1.P1
- net D8: now also BTN8.1, JP1.8; no longer S2.P, S2.P1
- net GND: now also BTN7.2, BTN8.2, RA0.1, VCC-GND-5V.2; no longer S1.S, S1.S1, S2.S, S2.S1
- net VCC: now also VCC-GND-5V.1
Other:
- note added: "Pullup for A0"
- note added: "Use 8266 INPUT_PULLUP."
- moved on the sheet: GND, GND-VCC-GND, VCC
